Commit message: fix: 修复 urdf 渲染

File: public/models/fins/fins.urdf (robot description, URDF)
Before this commit: robot FINES, 2 links, 1 joints
Links:
- link base_lidar: mass 0.156854810446873 -> None; geometry visual mesh filename=package://meshes/mid360.glb
- link base_link: mass 5.77687472400627 -> None; geometry visual mesh filename=package://meshes/base_link.glb
Joints:
- joint lidar_joint: axis 0 0 0 -> (none); origin xyz=0 0.083 0.31 rpy=0 0 0 -> xyz=0.057 0.083 0.31 rpy=3.14 2.3038346 3.14
