Commit message: perf: 使用 webworker 进行性能优化

File: public/models/wheelchair/wheelchair.urdf (robot description, URDF)
Before this commit: robot wheel_chair, 3 links, 2 joints
Links:
- removed link livox_frame_192_168_1_187
- removed link livox_frame_192_168_1_198
- added link main_lidar; visual mesh filename=package://meshes/mid360.glb
- added link sub_lidar; visual mesh filename=package://meshes/mid360.glb
Joints:
- removed joint livox_frame_192_168_1_187
- removed joint livox_frame_192_168_1_198
- added joint main_lidar: type fixed, parent base_link, child main_lidar, origin xyz=0.54961 0.23901 0.19335 rpy=0.0209 0.22689 -0.00698
- added joint sub_lidar: type fixed, parent base_link, child sub_lidar, origin xyz=0.54961 -0.23901 0.16335 rpy=-0.02269 0.22689 0.01396
